Commit message: update gazebo

File: Lemon_minibot_core/gazebo/minibot_Exported/minibot/minibot.URDF (robot description, URDF)
Before this commit: robot minibot, 4 links, 3 joints
Links:
- removed link l_whee;
- added link l_whee, mass 0.0714319766280304; collision mesh filename=package://minibot/collisionSTL/l_whee.STL; visual mesh filename=package://minibot/visualSTL/l_whee.STL
- link base: mass 0.00112497656106423 -> 0.000421866210399086
Joints:
- removed joint base-l_whee;
- added joint base-l_whee: type continuous, parent base, child l_whee, origin xyz=-0.0930787246278284 -0.0033654103350226 0.278465383032101 rpy=0 0 0, axis -1 -5.50460220501117E-15 4.19506831259459E-15
