Commit message: gazebo launch

File: lemon_minibot_core/gazebo/minibot_Exported/minibot/minibot.URDF (robot description, URDF)
Before this commit: robot minibot, 4 links, 3 joints
Links:
- removed link l_whee;
- added link l_whee, mass 0.0714319766280304; collision mesh filename=package://lemon_minibot_core/gazebo/minibot_Exported/minibo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; visual mesh filename=package://lemon_minibot_core/gazebo/minibot_Exported/minibo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
- link ball: geometry collision mesh filename=package://lemon_minibot_core/gazebo/minibot_Exported/minibo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; visual mesh filename=package://lemon_minibot_core/gazebo/minibot_Exported/minibo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
- link base: geometry collision mesh filename=package://lemon_minibot_core/gazebo/minibot_Exported/minibo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; visual mesh filename=package://lemon_minibot_core/gazebo/minibot_Exported/minibo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
- link r_wheel: geometry collision mesh filename=package://lemon_minibot_core/gazebo/minibot_Exported/minibo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; visual mesh filename=package://lemon_minibot_core/gazebo/minibot_Exported/minibo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
Joints:
- removed joint base-l_whee;
- added joint base-l_whee: type continuous, parent base, child l_whee, origin xyz=-0.0930787246278284 -0.0033654103350226 0.278465383032101 rpy=0 0 0, axis -1 -5.50460220501117E-15 4.19506831259459E-15
