Commit message: gazebo test

File: gazebo/minibot/robots/minibot.xacro (robot description, xacro)
@@ -34,5 +34,5 @@
       </material>
     </visual>
-    <collision>
+    <collision name='caster_collision'>
       <origin
         xyz="0 0 0"
@@ -42,4 +42,14 @@
           filename="package://minibot/meshes/base_link.STL" />
       </geometry>
+      <surface>
+        <friction>
+          <ode>
+            <mu>0</mu>
+            <mu2>0</mu2>
+            <slip1>1.0</slip1>
+            <slip2>1.0</slip2>
+          </ode>
+        </friction>
+      </surface>
     </collision>
   </link>
