Commit message: up gazebo info & reme

File: gazebo/turtlebot3_description/urdf/turtlebot3_waffle_pi.gazebo.xacro (robot description, xacro)
@@ -8,20 +8,20 @@
   </gazebo>
   <gazebo reference="wheel_left_link">
-    <mu1>0.1</mu1>
-    <mu2>0.1</mu2>
-    <kp>500000.0</kp>
+    <mu1>0.5</mu1>
+    <mu2>0.5</mu2>
+    <kp>50000.0</kp>
     <kd>10.0</kd>
     <minDepth>0.001</minDepth>
-    <maxVel>0.1</maxVel>
+    <maxVel>0.05</maxVel>
     <fdir1>1 0 0</fdir1>
     <material>Gazebo/Green</material>
   </gazebo>
   <gazebo reference="wheel_right_link">
-    <mu1>0.1</mu1>
-    <mu2>0.1</mu2>
-    <kp>500000.0</kp>
+    <mu1>0.5</mu1>
+    <mu2>0.5</mu2>
+    <kp>50000.0</kp>
     <kd>10.0</kd>
     <minDepth>0.001</minDepth>
-    <maxVel>0.1</maxVel>
+    <maxVel>0.05</maxVel>
     <fdir1>1 0 0</fdir1>
     <material>Gazebo/Green</material>
@@ -52,7 +52,7 @@
     <material>Gazebo/Grey</material>
   </gazebo>
-  <gazebo>
+  <!-- <gazebo>
     <plugin name="turtlebot3_waffle_pi_controller" filename="libgazebo_ros_diff_drive.so">
-      <commandTopic>cmd_vel</commandTopic>
+      <commandTopic>car/cmd_vel</commandTopic>
       <odometryTopic>odom</odometryTopic>
       <odometryFrame>odom</odometryFrame>
@@ -65,13 +65,30 @@
       <legacyMode>false</legacyMode>
       <updateRate>30</updateRate>
+      <leftJoint>wheel_right_joint</leftJoint>
+      <rightJoint>wheel_left_joint</rightJoint>
+      <wheelSeparation>0.287</wheelSeparation>
+      <wheelDiameter>0.066</wheelDiameter>
+      <wheelAcceleration>0.2</wheelAcceleration>
+      <wheelTorque>1</wheelTorque>
+      <rosDebugLevel>na</rosDebugLevel>
+    </plugin>
+</gazebo> -->
+<gazebo>
+    <plugin name="turtlebot3_waffle_pi_controller" filename="libgazebo_ros_diff_drive.so">
+      <legacyMode>false</legacyMode>
+      <alwaysOn>true</alwaysOn>
+      <updateRate>10</updateRate>
       <leftJoint>wheel_left_joint</leftJoint>
       <rightJoint>wheel_right_joint</rightJoint>
-      <wheelSeparation>0.287</wheelSeparation>
+      <wheelSeparation>0.28</wheelSeparation>
       <wheelDiameter>0.066</wheelDiameter>
-      <wheelAcceleration>1</wheelAcceleration>
-      <wheelTorque>10</wheelTorque>
-      <rosDebugLevel>na</rosDebugLevel>
+      <torque>1</torque>
+      <commandTopic>car/cmd_vel</commandTopic>
+      <odometryTopic>odom</odometryTopic>
+      <odometryFrame>odom</odometryFrame>
+      <robotBaseFrame>base_footprint</robotBaseFrame>
+      <robotBaseFrame>chassis</robotBaseFrame>
     </plugin>
-  </gazebo>
+</gazebo>
   <gazebo>
     <plugin name="imu_plugin" filename="libgazebo_ros_imu.so">

File: gazebo/turtlebot3_description/urdf/turtlebot3_waffle_pi.urdf.xacro (robot description, xacro)
@@ -25,5 +25,5 @@
     <inertial>
       <origin xyz="0 0 0" rpy="0 0 0"/>
-      <mass value="1.3729096e+00"/>
+      <mass value="1"/>
       <inertia ixx="8.7002718e-03" ixy="-4.7576583e-05" ixz="1.1160499e-04"
                iyy="8.6195418e-03" iyz="-3.5422299e-06"
@@ -53,5 +53,5 @@
     <inertial>
       <origin xyz="0 0 0" />
-      <mass value="2.8498940e-02" />
+      <mass value="0.1" />
       <inertia ixx="1.1175580e-05" ixy="-4.2369783e-11" ixz="-5.9381719e-09"
                iyy="1.1192413e-05" iyz="-1.4400107e-11"
@@ -81,5 +81,5 @@
     <inertial>
       <origin xyz="0 0 0" />
-      <mass value="2.8498940e-02" />
+      <mass value="0.1" />
       <inertia ixx="1.1175580e-05" ixy="-4.2369783e-11" ixz="-5.9381719e-09"
                iyy="1.1192413e-05" iyz="-1.4400107e-11"
