Commit message: ar in gazebo success

File: gazebo/turtlebot3_copy/urdf/turtlebot3_waffle_pi.gazebo.xacro (robot description, xacro)
@@ -151,28 +151,27 @@
     </sensor>
   </gazebo>
-<!--link : https://www.raspberrypi.org/documentation/hardware/camera/-->
-  <gazebo reference="camera_rgb_frame">
-    <sensor type="camera" name="Pi Camera">
-      <always_on>true</always_on>
-      <visualize>$(arg camera_visual)</visualize>
-      <camera>
-          <horizontal_fov>1.085595</horizontal_fov>
-          <image>
-              <width>640</width>
-              <height>480</height>
-              <format>R8G8B8</format>
-          </image>
-          <clip>
-              <near>0.03</near>
-              <far>100</far>
-          </clip>
+ <gazebo reference="camera_rgb_frame">
+    <material>Gazebo/Green</material>
+    <sensor type="camera" name="camera1">
+      <update_rate>30.0</update_rate>
+      <camera name="head">
+        <horizontal_fov>1.3962634</horizontal_fov>
+        <image>
+          <width>640</width>
+          <height>480</height>
+          <format>R8G8B8</format>
+        </image>
+        <clip>
+          <near>0.02</near>
+          <far>300</far>
+        </clip>
       </camera>
       <plugin name="camera_controller" filename="libgazebo_ros_camera.so">
         <alwaysOn>true</alwaysOn>
-        <updateRate>30.0</updateRate>
-        <cameraName>camera</cameraName>
-        <frameName>camera_rgb_optical_frame</frameName>
-        <imageTopicName>rgb/image_raw</imageTopicName>
-        <cameraInfoTopicName>rgb/camera_info</cameraInfoTopicName>
+        <updateRate>0.0</updateRate>
+        <cameraName>usb_cam</cameraName>
+        <imageTopicName>image_raw</imageTopicName>
+        <cameraInfoTopicName>camera_info</cameraInfoTopicName>
+        <frameName>camera</frameName>
         <hackBaseline>0.07</hackBaseline>
         <distortionK1>0.0</distortionK1>
@@ -183,4 +182,4 @@
       </plugin>
     </sensor>
-  </gazebo>
+</gazebo>
 </robot>

Commit message: angle fix

File: gazebo/turtlebot3_copy/urdf/turtlebot3_waffle_pi.gazebo.xacro (robot description, xacro)
@@ -154,4 +154,5 @@
     <material>Gazebo/Green</material>
     <sensor type="camera" name="camera1">
+      <pose>0 0 0 0 0 0</pose>
       <update_rate>30.0</update_rate>
       <camera name="head">

File: gazebo/turtlebot3_copy/urdf/turtlebot3_waffle_pi.urdf.xacro (robot description, xacro)
@@ -167,5 +167,5 @@
   <link name="camera_link">
     <collision>
-      <origin xyz="0.005 0.011 0.013" rpy="0 0 0"/>
+      <origin xyz="0.005 0.011 0.013" rpy="0 0 0"/> <!--xyz="0.005 0.011 0.013"-->
       <geometry>
         <box size="0.015 0.030 0.027"/>
